File: BatReservPwr.kicad_sch (KiCad schematic)
At the start: 9 parts, among them J8 Bat, Q1 IRLML6402, U4 MCP73831/2

Commit message: Ready for production
Parts:
- D2: descr (none) -> Low Vf
Other:
- title: (none) -> Universal board.  ESP-C3
- moved on the sheet: C8, D2, D4, J8, Q1
