File: PowerSupply.kicad_sch (KiCad schematic)
At the start: 20 parts, among them J4 220V, J7 USB_C_Receptacle_PowerOnly_6P, U2 BP2525F, U3 LP5907MFX-3.3

Commit message: Ready for production
Other:
- title: (none) -> Universal board.  ESP-C3
Changed lines of the file:
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@@
 	(paper "A4")
 	(title_block
+		(title "Universal board.  ESP-C3")
 		(date "2023-10-01")
 		(rev "12")
@@
 		(shape output)
 		(at 150.495 55.88 0)
+		(effects
+			(font
+				(size 1.27 1.27)
+			)
+			(justify left)
+		)
+	)
+	(hierarchical_label "+3V3"
+		(shape output)
+		(at 212.725 140.97 0)
 		(effects
 			(font
@@
 	)
 	(symbol
+		(lib_name "+5V_1")
 		(lib_id "power:+5V")
 		(at 267.97 25.4 180)
@@
 			)
 		)
-		(property "Description" ""
+		(property "Description" "Power symbol creates a global label with name \"+5V\""
 			(at 267.97 25.4 0)
 			(effects
