File: SMHome_UniversalRound_ESP32_C3_Mini_v3.kicad_pcb (KiCad board)
At the start: 2 copper layers, 48 x 45.6 mm, 58 parts, among them J1 K128_P3, J2 K128_P4, J3 Disp, J4 220V, J5 K128_P3, J6 JST SH, J7 USB_C_Receptacle_PowerOnly_6P, J8 Bat, Q1 IRLML6402, U1 ESP32 C3 Pro Mini, U2 BP2525F, U3 LP5907MFX-3.3, U4 MCP73831/2

Commit message: Ready for production
Parts:
- moved J8 2.28 mm to (159.2, 120.8), turned to -90 degrees
Routing:
- net Net-(J8-Pin_2): track 37.6 -> 46.1 mm
- net GND: track 200.4 -> 204.6 mm
