File: SMHome_UniversalRound_ESP32_C3_Mini_v3.kicad_sch (KiCad schematic)
At the start: 11 parts, among them J3 Disp, J6 JST SH, U1 ESP32 C3 Pro Mini

Commit message: Ready for production
Parts:
- TP2, TP3, TP4, TP5: now left out of the parts list
Connections:
- no-connect marks 0 -> 1
Other:
- title: Smart home relay board. -> Universal board.  ESP-C3
